Commit message: Moveble Mobile Base

File: urdf/mra.xacro (robot description, xacro)
@@ -89,5 +89,5 @@
 				<origin xyz="0 0 0" rpy="${-reflect*pi/2} 0 0"/>
 				<geometry>
-					<mesh filename="${mesh_path}" scale="0.01 0.01 0.01"/>
+					<cylinder radius="0.06" length="0.025"/>
 				</geometry>
 				<surface>
@@ -106,5 +106,5 @@
 			<parent link="${parent}"/>
 			<child link="wheel_${suffix}"/>
-			<origin xyz="-0.05 ${reflect*0.14} 0.05" rpy="0 0 0"/>
+			<origin xyz="-0.04 ${reflect*0.13} 0.05" rpy="0 0 0"/>
 			<axis xyz="0 1 0"/>
 			<!--limit velocity="4.8" effort="1" lower="${-pi}" upper="${pi}" /-->
@@ -114,9 +114,8 @@
 			<actuator name="$wheel_${suffix}_motor">
 				<mechanicalReduction>1</mechanicalReduction>
-				<hardwareInterface>EffortJointInterface</hardwareInterface>
+				<hardwareInterface>VelocityJointInterface</hardwareInterface>
 			</actuator>
 			<joint name="wheel_${suffix}_joint">
-				<hardwareInterface>PositionJointInterface</hardwareInterface>
-				<hardwareInterface>EffortJointInterface</hardwareInterface>
+				<hardwareInterface>hardware_interface/VelocityJointInterface</hardwareInterface>
 			</joint>
 		</transmission>
@@ -134,7 +133,7 @@
 		</visual>
 		<collision>
-			<origin xyz="0 0 0" rpy="0 0 0"/>
+			<origin xyz="0 0 0.075" rpy="0 0 0"/>
 			<geometry>
-				<mesh filename="package://innomech/meshes/base_link2.stl" scale="0.01 0.01 0.01"/>
+				<box size="0.2 0.2 0.14" />
 			</geometry>
 		</collision>
@@ -152,5 +151,5 @@
 			<origin xyz="0 0 0" rpy="0 0 0"/>
 			<geometry>
-				<sphere radius="0.01"/>
+				<sphere radius="0.005"/>
 			</geometry>
 		</collision>
@@ -160,7 +159,7 @@
 		<parent link="base_link"/>
 		<child link="point_wheel"/>
-		<origin xyz="0.08 0.0 -0.0025" rpy="0 0 0"/>
-		<axis xyz="1 1 1"/>
-		<limit effort="30" velocity="1.0"/>
+		<origin xyz="0.08 0.0 -0.0035" rpy="0 0 0"/>
+		<axis xyz="1 1 0"/>
+		<limit effort="1" velocity="10.0"/>
 	</joint>
 	<!-- Left Wheel -->

Commit message: Add Joystick Control

File: urdf/mra.xacro (robot description, xacro)
@@ -138,5 +138,5 @@
 			</geometry>
 		</collision>
-		<xacro:default_inertial mass="1.488" ixx="0.01143272" ixy="0.000016903" ixz="-0.000443487" iyy="0.000016903" iyz="-0.000443487" izz="-0.000443487"/>
+		<xacro:default_inertial mass="1.488" ixx="0.1143272" ixy="0.000016903" ixz="-0.000443487" iyy="0.000016903" iyz="-0.000443487" izz="-0.000443487"/>
 	</link>
 	<link name="point_wheel">
@@ -151,5 +151,5 @@
 			<origin xyz="0 0 0" rpy="0 0 0"/>
 			<geometry>
-				<sphere radius="0.005"/>
+				<sphere radius="0.0025"/>
 			</geometry>
 		</collision>
@@ -159,5 +159,5 @@
 		<parent link="base_link"/>
 		<child link="point_wheel"/>
-		<origin xyz="0.08 0.0 -0.0035" rpy="0 0 0"/>
+		<origin xyz="0.06 0.0 -0.0035" rpy="0 0 0"/>
 		<axis xyz="1 1 0"/>
 		<limit effort="1" velocity="10.0"/>

Commit message: Update Inertia

File: urdf/mra.xacro (robot description, xacro)
@@ -89,11 +89,11 @@
 				<origin xyz="0 0 0" rpy="${-reflect*pi/2} 0 0"/>
 				<geometry>
-					<cylinder radius="0.06" length="0.025"/>
+					<cylinder radius="0.057" length="0.025"/>
 				</geometry>
 				<surface>
 					<friction>
 						<ode>
-							<mu>0.05</mu>
-							<mu2>0.05</mu2>
+							<mu>0.5</mu>
+							<mu2>0.5</mu2>
 						</ode>
 					</friction>
@@ -135,9 +135,13 @@
 			<origin xyz="0 0 0.075" rpy="0 0 0"/>
 			<geometry>
-				<box size="0.2 0.2 0.14" />
+				<box size="0.2 0.18 0.14" />
 			</geometry>
 		</collision>
-		<xacro:default_inertial mass="1.488" ixx="0.1143272" ixy="0.000016903" ixz="-0.000443487" iyy="0.000016903" iyz="-0.000443487" izz="-0.000443487"/>
+		<!--0.0055676
+			0.0068975
+			0.0025451-->
+		<xacro:default_inertial mass="14.88" ixx="0.0073904" iyy="0.00992" izz="0.0073904"/>
 	</link>
+	<!-- Point Wheel -->
 	<link name="point_wheel">
 		<visual>
@@ -151,34 +155,37 @@
 			<origin xyz="0 0 0" rpy="0 0 0"/>
 			<geometry>
-				<sphere radius="0.0025"/>
+				<sphere radius="0.005"/>
 			</geometry>
 		</collision>
-		<xacro:default_inertial mass="0.01"/>
+		<xacro:default_inertial mass="0.05" ixx="0.0000144" ixy="0.0" ixz="0.0" iyy="0.0000144" iyz="0.0" izz="0.0000144"/>
 	</link>
 	<joint name="point_wheel_joint" type="continuous">
 		<parent link="base_link"/>
 		<child link="point_wheel"/>
-		<origin xyz="0.06 0.0 -0.0035" rpy="0 0 0"/>
+		<origin xyz="0.08 0.0 -0.0030" rpy="0 0 0"/>
 		<axis xyz="1 1 0"/>
-		<limit effort="1" velocity="10.0"/>
 	</joint>
+	<!-- Point Wheel -->
+	<!--0.0002285
+		0.0002285
+		0.000432-->
 	<!-- Left Wheel -->
-	<xacro:wheel_link suffix="left" parent="base_link" reflect="1" height="1" color="black" mesh_path="package://innomech/meshes/wheel_left_link2.stl" mass="0.240" ixx="0.000211589" ixy="0.0" ixz="0.0" iyy="0.0" iyz="0.0" izz="0.0"/>
+	<xacro:wheel_link suffix="left" parent="base_link" reflect="1" height="1" color="black" mesh_path="package://innomech/meshes/wheel_left_link2.stl" mass="2.40" ixx="0.0002285" ixy="0.0" ixz="0.0" iyy="0.0002285" iyz="0.0" izz="0.000432"/>
 	<!-- Left Wheel -->
 	<!-- Right Wheel -->
-	<xacro:wheel_link suffix="right" parent="base_link" reflect="-1" height="1" color="black" mesh_path="package://innomech/meshes/wheel_left_link2.stl" mass="0.240" ixx="0.000211589" ixy="0.0" ixz="0.0" iyy="0.0" iyz="0.0" izz="0.0"/>
+	<xacro:wheel_link suffix="right" parent="base_link" reflect="-1" height="1" color="black" mesh_path="package://innomech/meshes/wheel_left_link2.stl" mass="2.40" ixx="0.0002285" ixy="0.0" ixz="0.0" iyy="0.0002285" iyz="0.0" izz="0.000432"/>
 	<!-- Right Wheel -->
-	<!-- Link0 -->
-	<xacro:arm_link suffix="0" parent="base_link" reflect="1" height="0.25" color="red" mesh_path="package://innomech/meshes/mx-64t2.stl" mass="0.135" joint_type="revolute" lower_limit="${-pi}" upper_limit="${pi}" axis_x="0" axis_y="0" axis_z="1"/>
+	<!--Link0 -->
+	<xacro:arm_link suffix="0" parent="base_link" reflect="1" height="0.25" color="red" mesh_path="package://innomech/meshes/mx-64t2.stl" mass="1.35" joint_type="revolute" lower_limit="${-pi}" upper_limit="${pi}" axis_x="0" axis_y="0" axis_z="1"/>
 	<!-- Link0 -->
 	<!-- Link1 -->
-	<xacro:arm_link suffix="1" parent="armLink0" reflect="1" height="0.0" color="red" mesh_path="package://innomech/meshes/linked_mx_64t.stl" mass="0.168" joint_type="revolute" lower_limit="${-pi/4}" upper_limit="${pi/4}" axis_x="0" axis_y="1" axis_z="0" ixx="0.000208661" ixy="0.000000046" ixz="-0.000001178" iyy="0.000000046" iyz="-0.000001178" izz="-0.000001178"/>
+	<xacro:arm_link suffix="1" parent="armLink0" reflect="1" height="0.0" color="red" mesh_path="package://innomech/meshes/linked_mx_64t.stl" mass="1.68" joint_type="revolute" lower_limit="${-pi/4}" upper_limit="${pi/4}" axis_x="0" axis_y="1" axis_z="0" ixx="0.000208661" ixy="0.000000046" ixz="-0.000001178" iyy="0.000000046" iyz="-0.000001178" izz="-0.000001178"/>
 	<!-- Link1 -->
 	<!-- Link2 -->
-	<xacro:arm_link suffix="2" parent="armLink1" reflect="1" height="0.12" color="green" mesh_path="package://innomech/meshes/linked_mx_64t.stl" mass="0.168" joint_type="revolute" lower_limit="${-pi/4}" upper_limit="${pi/4}" axis_x="0" axis_y="1" axis_z="0" ixx="0.000208661" ixy="0.000000046" ixz="-0.000001178" iyy="0.000000046" iyz="-0.000001178" izz="-0.000001178"/>
+	<xacro:arm_link suffix="2" parent="armLink1" reflect="1" height="0.12" color="green" mesh_path="package://innomech/meshes/linked_mx_64t.stl" mass="1.68" joint_type="revolute" lower_limit="${-pi/4}" upper_limit="${pi/4}" axis_x="0" axis_y="1" axis_z="0" ixx="0.000208661" ixy="0.000000046" ixz="-0.000001178" iyy="0.000000046" iyz="-0.000001178" izz="-0.000001178"/>
 	<!-- Link2 -->
 	<!-- Link3 -->
-	<xacro:arm_link suffix="3" parent="armLink2" reflect="1" height="0.12" color="grey" mesh_path="package://innomech/meshes/linked_mx_64t.stl" mass="0.168" joint_type="revolute" lower_limit="${-pi/4}" upper_limit="${pi/4}" axis_x="0" axis_y="1" axis_z="0" ixx="0.000208661" ixy="0.000000046" ixz="-0.000001178" iyy="0.000000046" iyz="-0.000001178" izz="-0.000001178"/>
-	<!-- Link3 -->
+	<xacro:arm_link suffix="3" parent="armLink2" reflect="1" height="0.12" color="grey" mesh_path="package://innomech/meshes/linked_mx_64t.stl" mass="1.68" joint_type="revolute" lower_limit="${-pi/4}" upper_limit="${pi/4}" axis_x="0" axis_y="1" axis_z="0" ixx="0.000208661" ixy="0.000000046" ixz="-0.000001178" iyy="0.000000046" iyz="-0.000001178" izz="-0.000001178"/>
+	<!-- Link3 --> -->
 	<gazebo>
 		<plugin name="gazebo_ros_control" filename="libgazebo_ros_control.so">

Commit message: Update README.md

File: urdf/mra.xacro (robot description, xacro)
@@ -27,4 +27,8 @@
 	</material>
 	<!--Materials End-->
+	<xacro:property name="base_link_mass" value="1.488" />
+	<xacro:property name="arm_link_mass" value="0.168" />
+	<xacro:property name="wheel_mass" value="0.240" />
+	<xacro:property name="scale_" value="0.001" />
 	<!--MACROS START-->
 	<!--Inertial Macro-->
@@ -44,5 +48,5 @@
 				<geometry>
 					<!--mesh filename="package://innomech/meshes/linked_mx_64t.stl" scale="0.01 0.01 0.01"/-->
-					<mesh filename="${mesh_path}" scale="0.01 0.01 0.01"/>
+					<mesh filename="${mesh_path}" scale="${scale_} ${scale_} ${scale_}"/>
 				</geometry>
 				<material name="${color}"/>
@@ -51,5 +55,5 @@
 				<origin xyz="0 0 0" rpy="0 0 0"/>
 				<geometry>
-					<mesh filename="${mesh_path}" scale="0.01 0.01 0.01"/>
+					<mesh filename="${mesh_path}" scale="${scale_} ${scale_} ${scale_}"/>
 				</geometry>
 			</collision>
@@ -82,5 +86,5 @@
 				<geometry>
 					<!--mesh filename="package://innomech/meshes/wheel_left_link2.stl" scale="0.01 0.01 0.01"/-->
-					<mesh filename="${mesh_path}" scale="0.01 0.01 0.01"/>
+					<mesh filename="${mesh_path}" scale="${scale_} ${scale_} ${scale_}"/>
 				</geometry>
 				<material name="${color}"/>
@@ -89,5 +93,5 @@
 				<origin xyz="0 0 0" rpy="${-reflect*pi/2} 0 0"/>
 				<geometry>
-					<cylinder radius="0.057" length="0.025"/>
+					<cylinder radius="0.0057" length="0.0025"/>
 				</geometry>
 				<surface>
@@ -106,5 +110,5 @@
 			<parent link="${parent}"/>
 			<child link="wheel_${suffix}"/>
-			<origin xyz="-0.04 ${reflect*0.13} 0.05" rpy="0 0 0"/>
+			<origin xyz="-0.004 ${reflect*0.013} 0.005" rpy="0 0 0"/>
 			<axis xyz="0 1 0"/>
 			<!--limit velocity="4.8" effort="1" lower="${-pi}" upper="${pi}" /-->
@@ -128,12 +132,12 @@
 			<origin xyz="0 0 0" rpy="0 0 0"/>
 			<geometry>
-				<mesh filename="package://innomech/meshes/base_link2.stl" scale="0.01 0.01 0.01"/>
+				<mesh filename="package://innomech/meshes/base_link2.stl" scale="${scale_} ${scale_} ${scale_}"/>
 			</geometry>
 			<material name="white"/>
 		</visual>
 		<collision>
-			<origin xyz="0 0 0.075" rpy="0 0 0"/>
+			<origin xyz="0 0 0.0075" rpy="0 0 0"/>
 			<geometry>
-				<box size="0.2 0.18 0.14" />
+				<box size="0.02 0.018 0.014" />
 			</geometry>
 		</collision>
@@ -141,6 +145,6 @@
 			0.0068975
 			0.0025451-->
-		<xacro:default_inertial mass="14.88" ixx="0.0073904" iyy="0.00992" izz="0.0073904"/>
-	</link>
+			<xacro:default_inertial mass="${base_link_mass}" ixx="0.0073904" iyy="0.00992" izz="0.0073904"/>
+		</link>
 	<!-- Point Wheel -->
 	<link name="point_wheel">
@@ -148,5 +152,5 @@
 			<origin xyz="0 0 0" rpy="0 0 0"/>
 			<geometry>
-				<sphere radius="0.005"/>
+				<sphere radius="0.0005"/>
 			</geometry>
 			<material name="white"/>
@@ -155,41 +159,41 @@
 			<origin xyz="0 0 0" rpy="0 0 0"/>
 			<geometry>
-				<sphere radius="0.005"/>
+				<sphere radius="0.0005"/>
 			</geometry>
 		</collision>
 		<xacro:default_inertial mass="0.05" ixx="0.0000144" ixy="0.0" ixz="0.0" iyy="0.0000144" iyz="0.0" izz="0.0000144"/>
 	</link>
-	<joint name="point_wheel_joint" type="continuous">
-		<parent link="base_link"/>
-		<child link="point_wheel"/>
-		<origin xyz="0.08 0.0 -0.0030" rpy="0 0 0"/>
-		<axis xyz="1 1 0"/>
-	</joint>
-	<!-- Point Wheel -->
+		<joint name="point_wheel_joint" type="continuous">
+			<parent link="base_link"/>
+			<child link="point_wheel"/>
+			<origin xyz="0.008 0.0 -0.00030" rpy="0 0 0"/>
+			<axis xyz="1 1 0"/>
+		</joint>
+		<!-- Point Wheel -->
 	<!--0.0002285
 		0.0002285
 		0.000432-->
-	<!-- Left Wheel -->
-	<xacro:wheel_link suffix="left" parent="base_link" reflect="1" height="1" color="black" mesh_path="package://innomech/meshes/wheel_left_link2.stl" mass="2.40" ixx="0.0002285" ixy="0.0" ixz="0.0" iyy="0.0002285" iyz="0.0" izz="0.000432"/>
-	<!-- Left Wheel -->
-	<!-- Right Wheel -->
-	<xacro:wheel_link suffix="right" parent="base_link" reflect="-1" height="1" color="black" mesh_path="package://innomech/meshes/wheel_left_link2.stl" mass="2.40" ixx="0.0002285" ixy="0.0" ixz="0.0" iyy="0.0002285" iyz="0.0" izz="0.000432"/>
-	<!-- Right Wheel -->
-	<!--Link0 -->
-	<xacro:arm_link suffix="0" parent="base_link" reflect="1" height="0.25" color="red" mesh_path="package://innomech/meshes/mx-64t2.stl" mass="1.35" joint_type="revolute" lower_limit="${-pi}" upper_limit="${pi}" axis_x="0" axis_y="0" axis_z="1"/>
-	<!-- Link0 -->
-	<!-- Link1 -->
-	<xacro:arm_link suffix="1" parent="armLink0" reflect="1" height="0.0" color="red" mesh_path="package://innomech/meshes/linked_mx_64t.stl" mass="1.68" joint_type="revolute" lower_limit="${-pi/4}" upper_limit="${pi/4}" axis_x="0" axis_y="1" axis_z="0" ixx="0.000208661" ixy="0.000000046" ixz="-0.000001178" iyy="0.000000046" iyz="-0.000001178" izz="-0.000001178"/>
-	<!-- Link1 -->
-	<!-- Link2 -->
-	<xacro:arm_link suffix="2" parent="armLink1" reflect="1" height="0.12" color="green" mesh_path="package://innomech/meshes/linked_mx_64t.stl" mass="1.68" joint_type="revolute" lower_limit="${-pi/4}" upper_limit="${pi/4}" axis_x="0" axis_y="1" axis_z="0" ixx="0.000208661" ixy="0.000000046" ixz="-0.000001178" iyy="0.000000046" iyz="-0.000001178" izz="-0.000001178"/>
-	<!-- Link2 -->
-	<!-- Link3 -->
-	<xacro:arm_link suffix="3" parent="armLink2" reflect="1" height="0.12" color="grey" mesh_path="package://innomech/meshes/linked_mx_64t.stl" mass="1.68" joint_type="revolute" lower_limit="${-pi/4}" upper_limit="${pi/4}" axis_x="0" axis_y="1" axis_z="0" ixx="0.000208661" ixy="0.000000046" ixz="-0.000001178" iyy="0.000000046" iyz="-0.000001178" izz="-0.000001178"/>
-	<!-- Link3 --> -->
-	<gazebo>
-		<plugin name="gazebo_ros_control" filename="libgazebo_ros_control.so">
-			<robotNamespace>/</robotNamespace>
-		</plugin>
-	</gazebo>
-</robot>
+		<!-- Left Wheel -->
+		<xacro:wheel_link suffix="left" parent="base_link" reflect="1" height="1" color="black" mesh_path="package://innomech/meshes/wheel_left_link2.stl" mass="${wheel_mass}" ixx="0.0002285" ixy="0.0" ixz="0.0" iyy="0.0002285" iyz="0.0" izz="0.000432"/>
+		<!-- Left Wheel -->
+		<!-- Right Wheel -->
+		<xacro:wheel_link suffix="right" parent="base_link" reflect="-1" height="1" color="black" mesh_path="package://innomech/meshes/wheel_left_link2.stl" mass="${wheel_mass}" ixx="0.0002285" ixy="0.0" ixz="0.0" iyy="0.0002285" iyz="0.0" izz="0.000432"/>
+		<!-- Right Wheel -->
+		<!--Link0 -->
+		<xacro:arm_link suffix="0" parent="base_link" reflect="1" height="0.025" color="red" mesh_path="package://innomech/meshes/mx-64t2.stl" mass="1.35" joint_type="revolute" lower_limit="${-pi}" upper_limit="${pi}" axis_x="0" axis_y="0" axis_z="1"/>
+		<!-- Link0 -->
+		<!-- Link1 -->
+		<xacro:arm_link suffix="1" parent="armLink0" reflect="1" height="0.0" color="red" mesh_path="package://innomech/meshes/linked_mx_64t.stl" mass="${arm_link_mass}" joint_type="revolute" lower_limit="${-pi/4}" upper_limit="${pi/4}" axis_x="0" axis_y="1" axis_z="0" ixx="0.000208661" ixy="0.000000046" ixz="-0.000001178" iyy="0.000000046" iyz="-0.000001178" izz="-0.000001178"/>
+		<!-- Link1 -->
+		<!-- Link2 -->
+		<xacro:arm_link suffix="2" parent="armLink1" reflect="1" height="0.012" color="green" mesh_path="package://innomech/meshes/linked_mx_64t.stl" mass="${arm_link_mass}" joint_type="revolute" lower_limit="${-pi/4}" upper_limit="${pi/4}" axis_x="0" axis_y="1" axis_z="0" ixx="0.000208661" ixy="0.000000046" ixz="-0.000001178" iyy="0.000000046" iyz="-0.000001178" izz="-0.000001178"/>
+		<!-- Link2 -->
+		<!-- Link3 -->
+		<xacro:arm_link suffix="3" parent="armLink2" reflect="1" height="0.012" color="grey" mesh_path="package://innomech/meshes/linked_mx_64t.stl" mass="${arm_link_mass}" joint_type="revolute" lower_limit="${-pi/4}" upper_limit="${pi/4}" axis_x="0" axis_y="1" axis_z="0" ixx="0.000208661" ixy="0.000000046" ixz="-0.000001178" iyy="0.000000046" iyz="-0.000001178" izz="-0.000001178"/>
+		<!-- Link3 --> -->
+		<gazebo>
+			<plugin name="gazebo_ros_control" filename="libgazebo_ros_control.so">
+				<robotNamespace>/</robotNamespace>
+			</plugin>
+		</gazebo>
+	</robot>
