Commit message: Update robot_controller

File: urdf/mra.xacro (robot description, xacro)
@@ -27,8 +27,4 @@
 	</material>
 	<!--Materials End-->
-	<xacro:property name="base_link_mass" value="1.488" />
-	<xacro:property name="arm_link_mass" value="0.168" />
-	<xacro:property name="wheel_mass" value="0.240" />
-	<xacro:property name="scale_" value="0.001" />
 	<!--MACROS START-->
 	<!--Inertial Macro-->
@@ -48,5 +44,5 @@
 				<geometry>
 					<!--mesh filename="package://innomech/meshes/linked_mx_64t.stl" scale="0.01 0.01 0.01"/-->
-					<mesh filename="${mesh_path}" scale="${scale_} ${scale_} ${scale_}"/>
+					<mesh filename="${mesh_path}" scale="0.01 0.01 0.01"/>
 				</geometry>
 				<material name="${color}"/>
@@ -55,5 +51,5 @@
 				<origin xyz="0 0 0" rpy="0 0 0"/>
 				<geometry>
-					<mesh filename="${mesh_path}" scale="${scale_} ${scale_} ${scale_}"/>
+					<mesh filename="${mesh_path}" scale="0.01 0.01 0.01"/>
 				</geometry>
 			</collision>
@@ -86,5 +82,5 @@
 				<geometry>
 					<!--mesh filename="package://innomech/meshes/wheel_left_link2.stl" scale="0.01 0.01 0.01"/-->
-					<mesh filename="${mesh_path}" scale="${scale_} ${scale_} ${scale_}"/>
+					<mesh filename="${mesh_path}" scale="0.01 0.01 0.01"/>
 				</geometry>
 				<material name="${color}"/>
@@ -93,5 +89,5 @@
 				<origin xyz="0 0 0" rpy="${-reflect*pi/2} 0 0"/>
 				<geometry>
-					<cylinder radius="0.0057" length="0.0025"/>
+					<cylinder radius="0.057" length="0.025"/>
 				</geometry>
 				<surface>
@@ -110,5 +106,5 @@
 			<parent link="${parent}"/>
 			<child link="wheel_${suffix}"/>
-			<origin xyz="-0.004 ${reflect*0.013} 0.005" rpy="0 0 0"/>
+			<origin xyz="-0.04 ${reflect*0.13} 0.05" rpy="0 0 0"/>
 			<axis xyz="0 1 0"/>
 			<!--limit velocity="4.8" effort="1" lower="${-pi}" upper="${pi}" /-->
@@ -132,19 +128,16 @@
 			<origin xyz="0 0 0" rpy="0 0 0"/>
 			<geometry>
-				<mesh filename="package://innomech/meshes/base_link2.stl" scale="${scale_} ${scale_} ${scale_}"/>
+				<mesh filename="package://innomech/meshes/base_link2.stl" scale="0.01 0.01 0.01"/>
 			</geometry>
 			<material name="white"/>
 		</visual>
 		<collision>
-			<origin xyz="0 0 0.0075" rpy="0 0 0"/>
+			<origin xyz="0 0 0.075" rpy="0 0 0"/>
 			<geometry>
-				<box size="0.02 0.018 0.014" />
+				<box size="0.2 0.18 0.14" />
 			</geometry>
 		</collision>
-		<!--0.0055676
-			0.0068975
-			0.0025451-->
-			<xacro:default_inertial mass="${base_link_mass}" ixx="0.0073904" iyy="0.00992" izz="0.0073904"/>
-		</link>
+		<xacro:default_inertial mass="1.488" ixx="0.0073904" iyy="0.00992" izz="0.0073904"/>
+	</link>
 	<!-- Point Wheel -->
 	<link name="point_wheel">
@@ -152,5 +145,5 @@
 			<origin xyz="0 0 0" rpy="0 0 0"/>
 			<geometry>
-				<sphere radius="0.0005"/>
+				<sphere radius="0.005"/>
 			</geometry>
 			<material name="white"/>
@@ -159,41 +152,38 @@
 			<origin xyz="0 0 0" rpy="0 0 0"/>
 			<geometry>
-				<sphere radius="0.0005"/>
+				<sphere radius="0.005"/>
 			</geometry>
 		</collision>
 		<xacro:default_inertial mass="0.05" ixx="0.0000144" ixy="0.0" ixz="0.0" iyy="0.0000144" iyz="0.0" izz="0.0000144"/>
 	</link>
-		<joint name="point_wheel_joint" type="continuous">
-			<parent link="base_link"/>
-			<child link="point_wheel"/>
-			<origin xyz="0.008 0.0 -0.00030" rpy="0 0 0"/>
-			<axis xyz="1 1 0"/>
-		</joint>
-		<!-- Point Wheel -->
-	<!--0.0002285
-		0.0002285
-		0.000432-->
-		<!-- Left Wheel -->
-		<xacro:wheel_link suffix="left" parent="base_link" reflect="1" height="1" color="black" mesh_path="package://innomech/meshes/wheel_left_link2.stl" mass="${wheel_mass}" ixx="0.0002285" ixy="0.0" ixz="0.0" iyy="0.0002285" iyz="0.0" izz="0.000432"/>
-		<!-- Left Wheel -->
-		<!-- Right Wheel -->
-		<xacro:wheel_link suffix="right" parent="base_link" reflect="-1" height="1" color="black" mesh_path="package://innomech/meshes/wheel_left_link2.stl" mass="${wheel_mass}" ixx="0.0002285" ixy="0.0" ixz="0.0" iyy="0.0002285" iyz="0.0" izz="0.000432"/>
-		<!-- Right Wheel -->
-		<!--Link0 -->
-		<xacro:arm_link suffix="0" parent="base_link" reflect="1" height="0.025" color="red" mesh_path="package://innomech/meshes/mx-64t2.stl" mass="1.35" joint_type="revolute" lower_limit="${-pi}" upper_limit="${pi}" axis_x="0" axis_y="0" axis_z="1"/>
-		<!-- Link0 -->
-		<!-- Link1 -->
-		<xacro:arm_link suffix="1" parent="armLink0" reflect="1" height="0.0" color="red" mesh_path="package://innomech/meshes/linked_mx_64t.stl" mass="${arm_link_mass}" joint_type="revolute" lower_limit="${-pi/4}" upper_limit="${pi/4}" axis_x="0" axis_y="1" axis_z="0" ixx="0.000208661" ixy="0.000000046" ixz="-0.000001178" iyy="0.000000046" iyz="-0.000001178" izz="-0.000001178"/>
-		<!-- Link1 -->
-		<!-- Link2 -->
-		<xacro:arm_link suffix="2" parent="armLink1" reflect="1" height="0.012" color="green" mesh_path="package://innomech/meshes/linked_mx_64t.stl" mass="${arm_link_mass}" joint_type="revolute" lower_limit="${-pi/4}" upper_limit="${pi/4}" axis_x="0" axis_y="1" axis_z="0" ixx="0.000208661" ixy="0.000000046" ixz="-0.000001178" iyy="0.000000046" iyz="-0.000001178" izz="-0.000001178"/>
-		<!-- Link2 -->
-		<!-- Link3 -->
-		<xacro:arm_link suffix="3" parent="armLink2" reflect="1" height="0.012" color="grey" mesh_path="package://innomech/meshes/linked_mx_64t.stl" mass="${arm_link_mass}" joint_type="revolute" lower_limit="${-pi/4}" upper_limit="${pi/4}" axis_x="0" axis_y="1" axis_z="0" ixx="0.000208661" ixy="0.000000046" ixz="-0.000001178" iyy="0.000000046" iyz="-0.000001178" izz="-0.000001178"/>
-		<!-- Link3 --> -->
-		<gazebo>
-			<plugin name="gazebo_ros_control" filename="libgazebo_ros_control.so">
-				<robotNamespace>/</robotNamespace>
-			</plugin>
-		</gazebo>
-	</robot>
+	<joint name="point_wheel_joint" type="continuous">
+		<parent link="base_link"/>
+		<child link="point_wheel"/>
+		<origin xyz="0.08 0.0 -0.0030" rpy="0 0 0"/>
+		<axis xyz="1 1 0"/>
+	</joint>
+	<!-- Point Wheel -->
+	<!-- Left Wheel -->
+	<xacro:wheel_link suffix="left" parent="base_link" reflect="1" height="1" color="black" mesh_path="package://innomech/meshes/wheel_left_link2.stl" mass="0.240" ixx="0.0002285" ixy="0.0" ixz="0.0" iyy="0.0002285" iyz="0.0" izz="0.000432"/>
+	<!-- Left Wheel -->
+	<!-- Right Wheel -->
+	<xacro:wheel_link suffix="right" parent="base_link" reflect="-1" height="1" color="black" mesh_path="package://innomech/meshes/wheel_left_link2.stl" mass="0.240" ixx="0.0002285" ixy="0.0" ixz="0.0" iyy="0.0002285" iyz="0.0" izz="0.000432"/>
+	<!-- Right Wheel -->
+	<!--Link0 -->
+	<xacro:arm_link suffix="0" parent="base_link" reflect="1" height="0.25" color="red" mesh_path="package://innomech/meshes/mx-64t2.stl" mass="0.135" joint_type="revolute" lower_limit="${-pi}" upper_limit="${pi}" axis_x="0" axis_y="0" axis_z="1"/>
+	<!-- Link0 -->
+	<!-- Link1 -->
+	<xacro:arm_link suffix="1" parent="armLink0" reflect="1" height="0.0" color="red" mesh_path="package://innomech/meshes/linked_mx_64t.stl" mass="0.168" joint_type="revolute" lower_limit="${-pi/4}" upper_limit="${pi/4}" axis_x="0" axis_y="1" axis_z="0" ixx="0.000208661" ixy="0.000000046" ixz="-0.000001178" iyy="0.000000046" iyz="-0.000001178" izz="-0.000001178"/>
+	<!-- Link1 -->
+	<!-- Link2 -->
+	<xacro:arm_link suffix="2" parent="armLink1" reflect="1" height="0.12" color="green" mesh_path="package://innomech/meshes/linked_mx_64t.stl" mass="0.168" joint_type="revolute" lower_limit="${-pi/4}" upper_limit="${pi/4}" axis_x="0" axis_y="1" axis_z="0" ixx="0.000208661" ixy="0.000000046" ixz="-0.000001178" iyy="0.000000046" iyz="-0.000001178" izz="-0.000001178"/>
+	<!-- Link2 -->
+	<!-- Link3 -->
+	<xacro:arm_link suffix="3" parent="armLink2" reflect="1" height="0.12" color="grey" mesh_path="package://innomech/meshes/linked_mx_64t.stl" mass="0.168" joint_type="revolute" lower_limit="${-pi/4}" upper_limit="${pi/4}" axis_x="0" axis_y="1" axis_z="0" ixx="0.000208661" ixy="0.000000046" ixz="-0.000001178" iyy="0.000000046" iyz="-0.000001178" izz="-0.000001178"/>
+	<!-- Link3 --> -->
+	<gazebo>
+		<plugin name="gazebo_ros_control" filename="libgazebo_ros_control.so">
+			<robotNamespace>/</robotNamespace>
+		</plugin>
+	</gazebo>
+</robot>

Commit message: Automatically calculate mass matrixes

File: urdf/mra.xacro (robot description, xacro)
@@ -27,4 +27,9 @@
 	</material>
 	<!--Materials End-->
+	<xacro:property name="base_height" value="0.2" /> <!--x direction -->
+	<xacro:property name="base_width" value="0.2" /> <!--y direction -->
+	<xacro:property name="base_depth" value="0.14" /> <!--z direction -->
+	<xacro:property name="base_mass" value="1.488" /> <!--base mass -->
+	<xacro:property name="ball_wheel_radius" value="0.005" /> <!--base wheel radius -->
 	<!--MACROS START-->
 	<!--Inertial Macro-->
@@ -135,8 +140,11 @@
 			<origin xyz="0 0 0.075" rpy="0 0 0"/>
 			<geometry>
-				<box size="0.2 0.18 0.14" />
+				<box size="${base_height} ${base_width} ${base_depth}" />
 			</geometry>
 		</collision>
-		<xacro:default_inertial mass="1.488" ixx="0.0073904" iyy="0.00992" izz="0.0073904"/>
+		<xacro:default_inertial mass="${base_mass}"
+			ixx="${base_mass*(base_width*base_width+base_depth*base_depth)/12}"
+			iyy="${base_mass*(base_height*base_height+base_depth*base_depth)/12}"
+			izz="${base_mass*(base_width*base_width+base_height*base_height)/12}" />
 	</link>
 	<!-- Point Wheel -->
@@ -154,6 +162,17 @@
 				<sphere radius="0.005"/>
 			</geometry>
+			<surface>
+					<friction>
+						<ode>
+							<kp  value="10000000.0" />
+    						<kd  value="1.0" />
+						</ode>
+					</friction>
+				</surface>
 		</collision>
-		<xacro:default_inertial mass="0.05" ixx="0.0000144" ixy="0.0" ixz="0.0" iyy="0.0000144" iyz="0.0" izz="0.0000144"/>
+		<xacro:default_inertial mass="0.005"
+			ixx="${ball_wheel_radius*ball_wheel_radius*0.005*2/5}"
+			iyy="${ball_wheel_radius*ball_wheel_radius*0.005*2/5}"
+			izz="${ball_wheel_radius*ball_wheel_radius*0.005*2/5}"/>
 	</link>
 	<joint name="point_wheel_joint" type="continuous">
@@ -170,16 +189,4 @@
 	<xacro:wheel_link suffix="right" parent="base_link" reflect="-1" height="1" color="black" mesh_path="package://innomech/meshes/wheel_left_link2.stl" mass="0.240" ixx="0.0002285" ixy="0.0" ixz="0.0" iyy="0.0002285" iyz="0.0" izz="0.000432"/>
 	<!-- Right Wheel -->
-	<!--Link0 -->
-	<xacro:arm_link suffix="0" parent="base_link" reflect="1" height="0.25" color="red" mesh_path="package://innomech/meshes/mx-64t2.stl" mass="0.135" joint_type="revolute" lower_limit="${-pi}" upper_limit="${pi}" axis_x="0" axis_y="0" axis_z="1"/>
-	<!-- Link0 -->
-	<!-- Link1 -->
-	<xacro:arm_link suffix="1" parent="armLink0" reflect="1" height="0.0" color="red" mesh_path="package://innomech/meshes/linked_mx_64t.stl" mass="0.168" joint_type="revolute" lower_limit="${-pi/4}" upper_limit="${pi/4}" axis_x="0" axis_y="1" axis_z="0" ixx="0.000208661" ixy="0.000000046" ixz="-0.000001178" iyy="0.000000046" iyz="-0.000001178" izz="-0.000001178"/>
-	<!-- Link1 -->
-	<!-- Link2 -->
-	<xacro:arm_link suffix="2" parent="armLink1" reflect="1" height="0.12" color="green" mesh_path="package://innomech/meshes/linked_mx_64t.stl" mass="0.168" joint_type="revolute" lower_limit="${-pi/4}" upper_limit="${pi/4}" axis_x="0" axis_y="1" axis_z="0" ixx="0.000208661" ixy="0.000000046" ixz="-0.000001178" iyy="0.000000046" iyz="-0.000001178" izz="-0.000001178"/>
-	<!-- Link2 -->
-	<!-- Link3 -->
-	<xacro:arm_link suffix="3" parent="armLink2" reflect="1" height="0.12" color="grey" mesh_path="package://innomech/meshes/linked_mx_64t.stl" mass="0.168" joint_type="revolute" lower_limit="${-pi/4}" upper_limit="${pi/4}" axis_x="0" axis_y="1" axis_z="0" ixx="0.000208661" ixy="0.000000046" ixz="-0.000001178" iyy="0.000000046" iyz="-0.000001178" izz="-0.000001178"/>
-	<!-- Link3 --> -->
 	<gazebo>
 		<plugin name="gazebo_ros_control" filename="libgazebo_ros_control.so">

Commit message: Fix Inertia Matrix  Calculations, Update Casterback Wheel
Inertia matrixes changed by formulation, now being calculated according to the design parameters.
Casterback wheel turned into a fixed joint with small Mu values.
Acceleration increased.
PID controller values increased to sharper movement.

File: urdf/mra.xacro (robot description, xacro)
@@ -29,7 +29,10 @@
 	<xacro:property name="base_height" value="0.2" /> <!--x direction -->
 	<xacro:property name="base_width" value="0.2" /> <!--y direction -->
-	<xacro:property name="base_depth" value="0.14" /> <!--z direction -->
+	<xacro:property name="base_depth" value="0.2" /> <!--z direction -->
 	<xacro:property name="base_mass" value="1.488" /> <!--base mass -->
 	<xacro:property name="ball_wheel_radius" value="0.005" /> <!--base wheel radius -->
+	<xacro:property name="wheel_radius" value="0.06" /> <!--wheel radius -->
+	<xacro:property name="wheel_thickness" value="0.03" /> <!--wheel thickness -->
+	<xacro:property name="wheel_mass" value="0.240" /> <!--wheel mass-->
 	<!--MACROS START-->
 	<!--Inertial Macro-->
@@ -99,4 +102,6 @@
 					<friction>
 						<ode>
+							<kp>1000000</kp>
+							<kd>1</kd>
 							<mu>0.5</mu>
 							<mu2>0.5</mu2>
@@ -105,5 +110,8 @@
 				</surface>
 			</collision>
-			<xacro:default_inertial mass="${mass}"/>
+			<xacro:default_inertial mass="${mass}"
+				ixx="${wheel_mass*(3*wheel_radius*wheel_radius*wheel_radius+wheel_thickness*wheel_thickness)/12}"
+				iyy="${wheel_mass*(3*wheel_radius*wheel_radius*wheel_radius+wheel_thickness*wheel_thickness)/12}"
+				izz="${wheel_mass*wheel_radius*wheel_radius/2}"/>
 		</link>
 		<!-- Joint-->
@@ -138,5 +146,5 @@
 		</visual>
 		<collision>
-			<origin xyz="0 0 0.075" rpy="0 0 0"/>
+			<origin xyz="0 0 0.1" rpy="0 0 0"/>
 			<geometry>
 				<box size="${base_height} ${base_width} ${base_depth}" />
@@ -163,11 +171,13 @@
 			</geometry>
 			<surface>
-					<friction>
-						<ode>
-							<kp  value="10000000.0" />
-    						<kd  value="1.0" />
-						</ode>
-					</friction>
-				</surface>
+				<friction>
+					<ode>
+						<mu>0.1</mu>
+						<mu2>0.1</mu2>
+						<kp  value="10000000.0" />
+						<kd  value="1.0" />
+					</ode>
+				</friction>
+			</surface>
 		</collision>
 		<xacro:default_inertial mass="0.005"
@@ -176,9 +186,9 @@
 			izz="${ball_wheel_radius*ball_wheel_radius*0.005*2/5}"/>
 	</link>
-	<joint name="point_wheel_joint" type="continuous">
-		<parent link="base_link"/>
-		<child link="point_wheel"/>
-		<origin xyz="0.08 0.0 -0.0030" rpy="0 0 0"/>
-		<axis xyz="1 1 0"/>
+	<joint name="point_wheel_joint" type="fixed">
+			<parent link="base_link"/>
+			<child link="point_wheel"/>
+			<origin xyz="0.08 0.0 -0.0030" rpy="0 0 0"/>
+			<axis xyz="1 1 0"/>
 	</joint>
 	<!-- Point Wheel -->

Commit message: Update Arm Inertia Matrix

File: urdf/mra.xacro (robot description, xacro)
@@ -35,4 +35,8 @@
 	<xacro:property name="wheel_thickness" value="0.03" /> <!--wheel thickness -->
 	<xacro:property name="wheel_mass" value="0.240" /> <!--wheel mass-->
+	<xacro:property name="arm_height" value="0.06" /> <!--x direction -->
+	<xacro:property name="arm_width" value="0.06" /> <!--y direction -->
+	<xacro:property name="arm_depth" value="0.10" /> <!--z direction -->
+	<xacro:property name="arm_mass" value="0.168" /> <!--arm mass -->
 	<!--MACROS START-->
 	<!--Inertial Macro-->
@@ -46,5 +50,5 @@
 	<!--Inertial Macro-->
 	<!--Arm Link Macro-->
-	<xacro:macro name="arm_link" params="suffix parent reflect height color mesh_path mass joint_type lower_limit upper_limit axis_x axis_y axis_z ixx:=1 ixy:=0 ixz:=0 iyy:=1 iyz:=0 izz:=1">
+	<xacro:macro name="arm_link" params="suffix parent reflect height color mesh_path mass joint_type lower_limit upper_limit axis_x axis_y axis_z ixx:=1 ixy:=0 ixz:=0 iyy:=1 iyz:=0 izz:=1 arm_width_ arm_height_ arm_depth_ motor=0" >
 		<link name="armLink${suffix}">
 			<visual>
@@ -57,7 +61,7 @@
 			</visual>
 			<collision>
-				<origin xyz="0 0 0" rpy="0 0 0"/>
-				<geometry>
-					<mesh filename="${mesh_path}" scale="0.01 0.01 0.01"/>
+				<origin xyz="0 0 ${(1-motor)*arm_depth_}" rpy="0 0 0"/>
+				<geometry>
+					<box size="${arm_width_} ${arm_height_} ${arm_depth_}" />
 				</geometry>
 			</collision>
@@ -199,4 +203,27 @@
 	<xacro:wheel_link suffix="right" parent="base_link" reflect="-1" height="1" color="black" mesh_path="package://innomech/meshes/wheel_left_link2.stl" mass="0.240" ixx="0.0002285" ixy="0.0" ixz="0.0" iyy="0.0002285" iyz="0.0" izz="0.000432"/>
 	<!-- Right Wheel -->
+	<!--Link0 -->
+	<xacro:arm_link suffix="0" parent="base_link" reflect="1" height="0.25" color="orange" mesh_path="package://innomech/meshes/mx-64t2.stl" mass="0.135" joint_type="revolute" lower_limit="${-pi}" upper_limit="${pi}" axis_x="0" axis_y="0" axis_z="1"
+		arm_width_="0.04" arm_height_="0.04" arm_depth_="0.04" motor="1.0"/>
+	<!-- Link0 -->
+	<!-- Link1 -->
+	<xacro:arm_link suffix="1" parent="armLink0" reflect="1" height="0.0" color="red" mesh_path="package://innomech/meshes/linked_mx_64t.stl" mass="0.168" joint_type="revolute" lower_limit="${-pi/4}" upper_limit="${pi/4}" axis_x="0" axis_y="1" axis_z="0"
+		ixx="${arm_mass*(arm_width*arm_width+arm_depth*arm_depth)/12}"
+		iyy="${arm_mass*(arm_height*arm_height+arm_depth*arm_depth)/12}"
+		izz="${arm_mass*(arm_width*arm_width+arm_height*arm_height)/12}"
+		arm_width_="${arm_width}" arm_height_="${arm_height}" arm_depth_="${arm_depth}"/>
+	<!-- Link1 -->
+	<!-- Link2 -->
+	<xacro:arm_link suffix="2" parent="armLink1" reflect="1" height="0.12" color="green" mesh_path="package://innomech/meshes/linked_mx_64t.stl" mass="0.168" joint_type="revolute" lower_limit="${-pi/4}" upper_limit="${pi/4}" axis_x="0" axis_y="1" axis_z="0" 	ixx="${arm_mass*(arm_width*arm_width+arm_depth*arm_depth)/12}"
+		iyy="${arm_mass*(arm_height*arm_height+arm_depth*arm_depth)/12}"
+		izz="${arm_mass*(arm_width*arm_width+arm_height*arm_height)/12}"
+		arm_width_="${arm_width}" arm_height_="${arm_height}" arm_depth_="${arm_depth}"/>
+	<!-- Link2 -->
+	<!-- Link3 -->
+	<xacro:arm_link suffix="3" parent="armLink2" reflect="1" height="0.12" color="grey" mesh_path="package://innomech/meshes/linked_mx_64t.stl" mass="0.168" joint_type="revolute" lower_limit="${-pi/4}" upper_limit="${pi/4}" axis_x="0" axis_y="1" axis_z="0" 	ixx="${arm_mass*(arm_width*arm_width+arm_depth*arm_depth)/12}"
+		iyy="${arm_mass*(arm_height*arm_height+arm_depth*arm_depth)/12}"
+		izz="${arm_mass*(arm_width*arm_width+arm_height*arm_height)/12}"
+		arm_width_="${arm_width}" arm_height_="${arm_height}" arm_depth_="${arm_depth}"/>
+	<!-- Link3 -->
 	<gazebo>
 		<plugin name="gazebo_ros_control" filename="libgazebo_ros_control.so">

Commit message: Update VelocityJointInterface with EffortJointInterface
Due to bug in Gazebo v 7.0 mentioned here https://github.com/ros-simulation/gazebo_ros_pkgs/issues/612 changed the velocity type joints with effort joint type.

File: urdf/mra.xacro (robot description, xacro)
@@ -80,7 +80,8 @@
 			<actuator name="$armLink${suffix}_motor">
 				<mechanicalReduction>1</mechanicalReduction>
+				<hardwareInterface>EffortJointInterface</hardwareInterface>
 			</actuator>
 			<joint name="${parent}_armLink${suffix}_joint">
-				<hardwareInterface>PositionJointInterface</hardwareInterface>
+				<hardwareInterface>EffortJointInterface</hardwareInterface>
 			</joint>
 		</transmission>
@@ -190,8 +191,45 @@
 			izz="${ball_wheel_radius*ball_wheel_radius*0.005*2/5}"/>
 	</link>
-	<joint name="point_wheel_joint" type="fixed">
+	<joint name="point_wheel_joint" type="continuous">
 			<parent link="base_link"/>
 			<child link="point_wheel"/>
-			<origin xyz="0.08 0.0 -0.0030" rpy="0 0 0"/>
+			<origin xyz="0.08 0.04 -0.0030" rpy="0 0 0"/>
+			<axis xyz="1 1 0"/>
+	</joint>
+	<!-- Point Wheel -->
+	<!-- Point Wheel 2-->
+	<link name="point_wheel_right">
+		<visual>
+			<origin xyz="0 0 0" rpy="0 0 0"/>
+			<geometry>
+				<sphere radius="0.005"/>
+			</geometry>
+			<material name="white"/>
+		</visual>
+		<collision>
+			<origin xyz="0 0 0" rpy="0 0 0"/>
+			<geometry>
+				<sphere radius="0.005"/>
+			</geometry>
+			<surface>
+				<friction>
+					<ode>
+						<mu>0.1</mu>
+						<mu2>0.1</mu2>
+						<kp  value="10000000.0" />
+						<kd  value="1.0" />
+					</ode>
+				</friction>
+			</surface>
+		</collision>
+		<xacro:default_inertial mass="0.005"
+			ixx="${ball_wheel_radius*ball_wheel_radius*0.005*2/5}"
+			iyy="${ball_wheel_radius*ball_wheel_radius*0.005*2/5}"
+			izz="${ball_wheel_radius*ball_wheel_radius*0.005*2/5}"/>
+	</link>
+	<joint name="point_wheel_right_joint" type="continuous">
+			<parent link="base_link"/>
+			<child link="point_wheel_right"/>
+			<origin xyz="0.08 -0.04 -0.0030" rpy="0 0 0"/>
 			<axis xyz="1 1 0"/>
 	</joint>
