Commit message: Update Mobile Base Control & Arm Control

File: urdf/mra.xacro (robot description, xacro)
@@ -29,5 +29,5 @@
 	<xacro:property name="base_height" value="0.2" /> <!--x direction -->
 	<xacro:property name="base_width" value="0.2" /> <!--y direction -->
-	<xacro:property name="base_depth" value="0.2" /> <!--z direction -->
+	<xacro:property name="base_depth" value="0.20" /> <!--z direction -->
 	<xacro:property name="base_mass" value="1.488" /> <!--base mass -->
 	<xacro:property name="ball_wheel_radius" value="0.005" /> <!--base wheel radius -->
@@ -50,5 +50,5 @@
 	<!--Inertial Macro-->
 	<!--Arm Link Macro-->
-	<xacro:macro name="arm_link" params="suffix parent reflect height color mesh_path mass joint_type lower_limit upper_limit axis_x axis_y axis_z ixx:=1 ixy:=0 ixz:=0 iyy:=1 iyz:=0 izz:=1 arm_width_ arm_height_ arm_depth_ motor=0" >
+	<xacro:macro name="arm_link" params="suffix parent reflect height color mesh_path mass joint_type lower_limit upper_limit axis_x axis_y axis_z ixx:=1 ixy:=0 ixz:=0 iyy:=1 iyz:=0 izz:=1 arm_width_ arm_height_ arm_depth_ motor=0 jointInterface=Position ">
 		<link name="armLink${suffix}">
 			<visual>
@@ -78,10 +78,9 @@
 		<transmission name="armLink${suffix}_transmission" type="SimpleTransmission">
 			<type>transmission_interface/SimpleTransmission</type>
-			<actuator name="$armLink${suffix}_motor">
-				<mechanicalReduction>1</mechanicalReduction>
-				<hardwareInterface>EffortJointInterface</hardwareInterface>
+			<actuator name="armLink${suffix}_motor">
+				<hardwareInterface>hardware_interface/${jointInterface}JointInterface</hardwareInterface>
 			</actuator>
 			<joint name="${parent}_armLink${suffix}_joint">
-				<hardwareInterface>EffortJointInterface</hardwareInterface>
+				<hardwareInterface>hardware_interface/${jointInterface}JointInterface</hardwareInterface>
 			</joint>
 		</transmission>
@@ -159,7 +158,7 @@
 			ixx="${base_mass*(base_width*base_width+base_depth*base_depth)/12}"
 			iyy="${base_mass*(base_height*base_height+base_depth*base_depth)/12}"
-			izz="${base_mass*(base_width*base_width+base_height*base_height)/12}" />
+			izz="${base_mass*(base_width*base_width+base_height*base_height)/24}" />
 	</link>
-	<!-- Point Wheel -->
+	<!-- Point Wheel 1-->
 	<link name="point_wheel">
 		<visual>
@@ -178,6 +177,6 @@
 				<friction>
 					<ode>
-						<mu>0.1</mu>
-						<mu2>0.1</mu2>
+						<mu>0.00001</mu>
+						<mu2>0.8</mu2>
 						<kp  value="10000000.0" />
 						<kd  value="1.0" />
@@ -194,45 +193,7 @@
 			<parent link="base_link"/>
 			<child link="point_wheel"/>
-			<origin xyz="0.08 0.04 -0.0030" rpy="0 0 0"/>
-			<axis xyz="1 1 0"/>
+			<origin xyz="0.08 0.0 -0.0030" rpy="0 0 0"/>
+			<axis xyz="1 0 0"/>
 	</joint>
-	<!-- Point Wheel -->
-	<!-- Point Wheel 2-->
-	<link name="point_wheel_right">
-		<visual>
-			<origin xyz="0 0 0" rpy="0 0 0"/>
-			<geometry>
-				<sphere radius="0.005"/>
-			</geometry>
-			<material name="white"/>
-		</visual>
-		<collision>
-			<origin xyz="0 0 0" rpy="0 0 0"/>
-			<geometry>
-				<sphere radius="0.005"/>
-			</geometry>
-			<surface>
-				<friction>
-					<ode>
-						<mu>0.1</mu>
-						<mu2>0.1</mu2>
-						<kp  value="10000000.0" />
-						<kd  value="1.0" />
-					</ode>
-				</friction>
-			</surface>
-		</collision>
-		<xacro:default_inertial mass="0.005"
-			ixx="${ball_wheel_radius*ball_wheel_radius*0.005*2/5}"
-			iyy="${ball_wheel_radius*ball_wheel_radius*0.005*2/5}"
-			izz="${ball_wheel_radius*ball_wheel_radius*0.005*2/5}"/>
-	</link>
-	<joint name="point_wheel_right_joint" type="continuous">
-			<parent link="base_link"/>
-			<child link="point_wheel_right"/>
-			<origin xyz="0.08 -0.04 -0.0030" rpy="0 0 0"/>
-			<axis xyz="1 1 0"/>
-	</joint>
-	<!-- Point Wheel -->
 	<!-- Left Wheel -->
 	<xacro:wheel_link suffix="left" parent="base_link" reflect="1" height="1" color="black" mesh_path="package://innomech/meshes/wheel_left_link2.stl" mass="0.240" ixx="0.0002285" ixy="0.0" ixz="0.0" iyy="0.0002285" iyz="0.0" izz="0.000432"/>
@@ -242,6 +203,6 @@
 	<!-- Right Wheel -->
 	<!--Link0 -->
-	<xacro:arm_link suffix="0" parent="base_link" reflect="1" height="0.25" color="orange" mesh_path="package://innomech/meshes/mx-64t2.stl" mass="0.135" joint_type="revolute" lower_limit="${-pi}" upper_limit="${pi}" axis_x="0" axis_y="0" axis_z="1"
-		arm_width_="0.04" arm_height_="0.04" arm_depth_="0.04" motor="1.0"/>
+	<xacro:arm_link suffix="0" parent="base_link" reflect="1" height="0.25" color="orange" mesh_path="package://innomech/meshes/mx-64t2.stl" mass="0.135" joint_type="revolute" lower_limit="${-pi/2}" upper_limit="${pi/2}" axis_x="0" axis_y="0" axis_z="1"
+		arm_width_="0.04" arm_height_="0.04" arm_depth_="0.04" motor="1.0" jointInterface="Position"/>
 	<!-- Link0 -->
 	<!-- Link1 -->

Commit message: Add Arm Lock, Gazebo Colors

File: urdf/mra.xacro (robot description, xacro)
@@ -26,4 +26,11 @@
 		<color rgba="${222/255} ${207/255} ${195/255} 1.0"/>
 	</material>
+	<gazebo reference="base_link"><material>Gazebo/Black</material></gazebo>
+	<gazebo reference="wheel_left"><material>Gazebo/Grey</material></gazebo>
+	<gazebo reference="wheel_right"><material>Gazebo/Grey</material></gazebo>
+	<gazebo reference="armLink0"><material>Gazebo/Orange</material></gazebo>
+	<gazebo reference="armLink1"><material>Gazebo/Orange</material></gazebo>
+	<gazebo reference="armLink2"><material>Gazebo/Orange</material></gazebo>
+	<gazebo reference="armLink3"><material>Gazebo/Orange</material></gazebo>
 	<!--Materials End-->
 	<xacro:property name="base_height" value="0.2" /> <!--x direction -->
